Commit message: Restoring local changes

File: components/arm/robotiq_gripper.urdf.xacro (robot description, xacro)
@@ -1,16 +1,19 @@
 <?xml version="1.0"?>
-<!-- This is the URDF file for Robotiq 2f 140 Gripper-->
+<!-- This is the URDF file for Robotiq 2f 85 Gripper-->
 <robot xmlns:xacro="http://www.ros.org/wiki/xacro" name="robotiq_gripper">
+            <!-- Get tf_prefix from parent scope -->
+            <xacro:arg name="tf_prefix" default="ur5e"/>
+            <xacro:property name="tf_prefix" value="$(arg tf_prefix)"/>
             <!-- ur_adapter for gripper-->
             <xacro:include filename="$(find robotiq_description)/urdf/ur_to_robotiq_adapter.urdf.xacro"/>
             <xacro:ur_to_robotiq
                 prefix=""
-                parent="$(arg tf_prefix)tool0"
-                child="neo_gripper_mount_link"
+                parent="${tf_prefix}tool0"
+                child="gripper_mount_link"
                 rotation="${pi/2}"
                 />
-            <!-- add gripper-->
-            <xacro:include filename="$(find robotiq_description)/urdf/robotiq_2f_140_macro.urdf.xacro"/>
-            <xacro:robotiq_gripper name="robotiq_gripper" prefix="" parent="neo_gripper_mount_link" include_ros2_control="true" sim_ignition="true">
+            <!-- add gripper - using 2F-85 model which is available-->
+            <xacro:include filename="$(find robotiq_description)/urdf/robotiq_2f_85_macro.urdf.xacro"/>
+            <xacro:robotiq_gripper name="robotiq_gripper" prefix="" parent="gripper_mount_link" use_fake_hardware="true">
                 <origin xyz="0 0 0" rpy="0 0 -${pi / 2}"/>
             </xacro:robotiq_gripper>

Commit message: Localization working

File: components/arm/robotiq_gripper.urdf.xacro (robot description, xacro)
@@ -9,6 +9,5 @@
             <xacro:ur_to_robotiq
                 prefix=""
-                parent="${tf_prefix}tool0"
-                child="gripper_mount_link"
+                connected_to="${tf_prefix}tool0"
                 rotation="${pi/2}"
                 />
@@ -18,3 +17,15 @@
                 <origin xyz="0 0 0" rpy="0 0 -${pi / 2}"/>
             </xacro:robotiq_gripper>
+            <!-- Gazebo plugin to publish gripper joint states -->
+            <gazebo>
+                <plugin name="gazebo_ros_joint_state_publisher" filename="libgazebo_ros_joint_state_publisher.so">
+                    <update_rate>30</update_rate>
+                    <joint_name>robotiq_85_left_knuckle_joint</joint_name>
+                    <joint_name>robotiq_85_right_knuckle_joint</joint_name>
+                    <joint_name>robotiq_85_left_inner_knuckle_joint</joint_name>
+                    <joint_name>robotiq_85_right_inner_knuckle_joint</joint_name>
+                    <joint_name>robotiq_85_left_finger_tip_joint</joint_name>
+                    <joint_name>robotiq_85_right_finger_tip_joint</joint_name>
+                </plugin>
+            </gazebo>
 </robot>

File: components/dynamixel/steve_pan_tilt.xacro (robot description, xacro)
@@ -4,5 +4,5 @@
   <xacro:include filename="$(find neo_simulation2)/components/dynamixel/dynamixel_bracket_fr12_h101.urdf.xacro" />
   <xacro:arg name="grasp_link_offset" default="0.11"/>
-  <xacro:macro name="steve_pan_tilt" params="parent name *origin">
++  <xacro:macro name="steve_pan_tilt" params="parent name">
     <!-- Pan motor -->
     <xacro:dynamixel_motor_XL-430 name="${name}_tilt_motor" parent="${parent}" motor_direction="-1" position_offset="0.065">

File: components/pan_tilt/pan_tilt_tower.urdf.xacro (robot description, xacro)
@@ -14,5 +14,5 @@
       <parent link="${parent_link}"/>
       <child link="pan_tilt_tower_base"/>
-      <origin xyz="-0.2 0 1.214" rpy="0 0 0" />
+      <origin xyz="-0.15 0 1.1" rpy="0 0 0" />
     </joint>
     <!-- Tower vertical support pole -->
@@ -37,7 +37,5 @@
     <!-- Include Dynamixel pan-tilt mechanism -->
     <xacro:include filename="$(find neo_simulation2)/components/dynamixel/steve_pan_tilt.xacro"/>
-    <xacro:steve_pan_tilt parent="pan_tilt_tower_base" name="pan_tilt">
-      <origin xyz="0.0 0.0 0.0" rpy="0 0 0"/>
-    </xacro:steve_pan_tilt>
+    <xacro:steve_pan_tilt parent="pan_tilt_tower_base" name="pan_tilt"/>
     <!-- ROS2 Control for Pan-Tilt -->
     <xacro:include filename="$(find neo_simulation2)/components/pan_tilt/pan_tilt.ros2_control.xacro"/>

Commit message: Fix3

File: components/arm/robotiq_gripper.urdf.xacro (robot description, xacro)
@@ -1,19 +1,18 @@
 <?xml version="1.0"?>
 <robot xmlns:xacro="http://www.ros.org/wiki/xacro" name="robotiq_gripper">
-            <xacro:arg name="tf_prefix" default="ur5e"/>
-            <xacro:property name="tf_prefix" value="$(arg tf_prefix)"/>
-            <xacro:include filename="$(find robotiq_description)/urdf/ur_to_robotiq_adapter.urdf.xacro"/>
-            <xacro:ur_to_robotiq
-                prefix=""
-                connected_to="${tf_prefix}tool0"
-                rotation="${pi/2}"
-                />
-            <xacro:include filename="$(find robotiq_description)/urdf/robotiq_2f_85_macro.urdf.xacro"/>
-            <xacro:robotiq_gripper
-                name="robotiq_gripper"
-                prefix=""
-                parent_link="gripper_mount_link"
-                use_fake_hardware="true">
-                <origin xyz="0 0 0" rpy="0 0 -${pi / 2}"/>
-            </xacro:robotiq_gripper>
+    <xacro:arg name="tf_prefix" default="ur5e"/>
+    <xacro:property name="tf_prefix" value="$(arg tf_prefix)"/>
+    <xacro:include filename="$(find robotiq_description)/urdf/ur_to_robotiq_adapter.urdf.xacro"/>
+    <xacro:ur_to_robotiq
+        prefix=""
+        connected_to="${tf_prefix}tool0"
+        rotation="${pi/2}"
+    />
+    <xacro:include filename="$(find robotiq_description)/urdf/robotiq_2f_85_macro.urdf.xacro"/>
+    <xacro:robotiq_gripper
+        name="robotiq_gripper"
+        prefix=""
+        use_fake_hardware="true">
+        <origin xyz="0 0 0" rpy="0 0 -${pi / 2}"/>
+    </xacro:robotiq_gripper>
 </robot>
