Commit message: Restructure

File: components/arm/ur_arm.urdf.xacro (robot description, xacro)
@@ -17,6 +17,6 @@
             <xacro:arg name="safety_k_position" default="20"/>
             <xacro:arg name="sim_gazebo" default="$(arg use_gazebo)" />
-            <xacro:arg name="simulation_controllers" default="$(find neo_simulation2)/configs/ur_config/$(arg arm_type)/ur_controllers.yaml"/>
-            <xacro:arg name="initial_positions_file" default="$(find neo_simulation2)/configs/ur_config/initial_joint_positions.yaml"/>
+            <xacro:arg name="simulation_controllers" default="$(find steve_simulation)/configs/ur_config/$(arg arm_type)/ur_controllers.yaml"/>
+            <xacro:arg name="initial_positions_file" default="$(find steve_simulation)/configs/ur_config/initial_joint_positions.yaml"/>
             <!-- parse initial positions as a dictionary -->
             <xacro:property
@@ -55,4 +55,4 @@
             </xacro:if>
             <!-- include wrist camera mount (dummy end-effector with camera) -->
-            <xacro:include filename="$(find neo_simulation2)/components/arm/wrist_camera_mount.urdf.xacro"/>
+            <xacro:include filename="$(find steve_simulation)/components/arm/wrist_camera_mount.urdf.xacro"/>
 </robot>

File: components/arm/wrist_camera_mount.urdf.xacro (robot description, xacro)
@@ -37,5 +37,5 @@
             </link>
             <!-- Include wrist camera -->
-            <xacro:include filename="$(find neo_simulation2)/components/cameras/wrist_d405.urdf.xacro"/>
+            <xacro:include filename="$(find steve_simulation)/components/cameras/wrist_d405.urdf.xacro"/>
             <xacro:wrist_d405 parent="dummy_end_effector" use_gazebo="$(arg use_gazebo)"/>
 </robot>

File: components/cameras/wrist_d405.urdf.xacro (robot description, xacro)
@@ -14,5 +14,5 @@
     <origin xyz="0 0 0" rpy="0 0 0"/>
     <geometry>
-      <mesh filename="package://neo_simulation2/robots/mmo_700/meshes/cameras/d405/UR5_LastJointSensor_D405_Psyonic.STL" scale="0.001 0.001 0.001"/>
+      <mesh filename="package://steve_simulation/robots/mmo_700/meshes/cameras/d405/UR5_LastJointSensor_D405_Psyonic.STL" scale="0.001 0.001 0.001"/>
     </geometry>
     <material name="grey"/>
@@ -41,5 +41,5 @@
     <origin xyz="0.01 0 0.01" rpy="0 1.57 0"/>
     <geometry>
-      <mesh filename="package://neo_simulation2/robots/mmo_700/meshes/cameras/d405/d405.stl" scale="0.001 0.001 0.001"/>
+      <mesh filename="package://steve_simulation/robots/mmo_700/meshes/cameras/d405/d405.stl" scale="0.001 0.001 0.001"/>
     </geometry>
     <material name="grey"/>

File: components/common_macro/mpo_cabinet_macro.xacro (robot description, xacro)
@@ -26,5 +26,5 @@
                 <origin rpy="${visual_rpy}" xyz="0 0 0"/>
                 <geometry>
-                    <mesh filename="package://neo_simulation2/robots/${neo_robot_name}/meshes/cabin.dae" scale="${model_scale}"/>
+                    <mesh filename="package://steve_simulation/robots/${neo_robot_name}/meshes/cabin.dae" scale="${model_scale}"/>
                 </geometry>
             </visual>
@@ -32,5 +32,5 @@
                 <origin rpy="${collision_rpy}" xyz="0 0 0"/>
                 <geometry>
-                    <mesh filename="package://neo_simulation2/robots/${neo_robot_name}/meshes/cabin.dae" scale="${model_scale}"/>
+                    <mesh filename="package://steve_simulation/robots/${neo_robot_name}/meshes/cabin.dae" scale="${model_scale}"/>
                 </geometry>
             </collision>

File: components/dynamixel/dynamixel_bracket_fr12_h101.urdf.xacro (robot description, xacro)
@@ -16,5 +16,5 @@
         <origin xyz="0 0 0" rpy="0 0 0" />
         <geometry>
-          <mesh filename="package://neo_simulation2/robots/mmo_700/meshes/cameras/dynamixel/dynamixel_bracket_fr12_h101.dae" scale="0.001 0.001 0.001" />
+          <mesh filename="package://steve_simulation/robots/mmo_700/meshes/cameras/dynamixel/dynamixel_bracket_fr12_h101.dae" scale="0.001 0.001 0.001" />
         </geometry>
       </visual>
@@ -22,5 +22,5 @@
         <origin xyz="0 0 0" rpy="0 0 0" />
         <geometry>
-          <mesh filename="package://neo_simulation2/robots/mmo_700/meshes/cameras/dynamixel/dynamixel_bracket_fr12_h101_convex_hull.dae" scale="0.001 0.001 0.001" />
+          <mesh filename="package://steve_simulation/robots/mmo_700/meshes/cameras/dynamixel/dynamixel_bracket_fr12_h101_convex_hull.dae" scale="0.001 0.001 0.001" />
         </geometry>
       </collision>

File: components/dynamixel/dynamixel_motor_xl-430.urdf.xacro (robot description, xacro)
@@ -1,6 +1,6 @@
 <?xml version="1.0"?>
 <robot xmlns:xacro="http://www.ros.org/wiki/xacro">
-  <xacro:include filename="$(find neo_simulation2)/components/dynamixel/dynamixel_motor_xl-430.gazebo.xacro" />
-  <xacro:include filename="$(find neo_simulation2)/components/dynamixel/dynamixel_motor_xl-430.transmission.xacro" />
+  <xacro:include filename="$(find steve_simulation)/components/dynamixel/dynamixel_motor_xl-430.gazebo.xacro" />
+  <xacro:include filename="$(find steve_simulation)/components/dynamixel/dynamixel_motor_xl-430.transmission.xacro" />
   <xacro:property name="M_PI" value="3.1415926535897931" />
   <xacro:macro name="dynamixel_motor_XL-430" params="parent name *origin motor_direction position_offset">
@@ -19,5 +19,5 @@
         <origin xyz="0 0 0.0" rpy="0 ${pi/2} 0" />
         <geometry>
-          <mesh filename="package://neo_simulation2/robots/mmo_700/meshes/cameras/dynamixel/dynamixel_motor_xl-430.dae" scale="0.001 0.001 0.001" />
+          <mesh filename="package://steve_simulation/robots/mmo_700/meshes/cameras/dynamixel/dynamixel_motor_xl-430.dae" scale="0.001 0.001 0.001" />
         </geometry>
       </visual>
@@ -25,5 +25,5 @@
         <origin xyz="0 0 0.0" rpy="0 ${M_PI/2} 0" />
         <geometry>
-          <mesh filename="package://neo_simulation2/robots/mmo_700/meshes/cameras/dynamixel/dynamixel_motor_xl-430_convex_hull.dae" scale="0.001 0.001 0.001" />
+          <mesh filename="package://steve_simulation/robots/mmo_700/meshes/cameras/dynamixel/dynamixel_motor_xl-430_convex_hull.dae" scale="0.001 0.001 0.001" />
         </geometry>
       </collision>

File: components/dynamixel/steve_pan_tilt.xacro (robot description, xacro)
@@ -1,6 +1,6 @@
 <?xml version="1.0"?>
 <robot xmlns:xacro="http://www.ros.org/wiki/xacro">
-  <xacro:include filename="$(find neo_simulation2)/components/dynamixel/dynamixel_motor_xl-430.urdf.xacro" />
-  <xacro:include filename="$(find neo_simulation2)/components/dynamixel/dynamixel_bracket_fr12_h101.urdf.xacro" />
+  <xacro:include filename="$(find steve_simulation)/components/dynamixel/dynamixel_motor_xl-430.urdf.xacro" />
+  <xacro:include filename="$(find steve_simulation)/components/dynamixel/dynamixel_bracket_fr12_h101.urdf.xacro" />
   <xacro:arg name="grasp_link_offset" default="0.11"/>
 +  <xacro:macro name="steve_pan_tilt" params="parent name">

File: components/pan_tilt/pan_tilt_tower.urdf.xacro (robot description, xacro)
@@ -36,11 +36,11 @@
     </link>
     <!-- Include Dynamixel pan-tilt mechanism -->
-    <xacro:include filename="$(find neo_simulation2)/components/dynamixel/steve_pan_tilt.xacro"/>
+    <xacro:include filename="$(find steve_simulation)/components/dynamixel/steve_pan_tilt.xacro"/>
     <xacro:steve_pan_tilt parent="pan_tilt_tower_base" name="pan_tilt"/>
     <!-- ROS2 Control for Pan-Tilt -->
-    <xacro:include filename="$(find neo_simulation2)/components/pan_tilt/pan_tilt.ros2_control.xacro"/>
+    <xacro:include filename="$(find steve_simulation)/components/pan_tilt/pan_tilt.ros2_control.xacro"/>
     <xacro:pan_tilt_ros2_control name="pan_tilt"/>
     <!-- Include L515 camera macro -->
-    <xacro:include filename="$(find neo_simulation2)/components/cameras/l515_simplified.urdf.xacro"/>
+    <xacro:include filename="$(find steve_simulation)/components/cameras/l515_simplified.urdf.xacro"/>
     <!-- L515 Camera mounted on pan bracket (follows both pan and tilt) -->
     <xacro:sensor_l515_simplified

File: robots/mmo_700/mmo_700.urdf.xacro (robot description, xacro)
@@ -22,8 +22,8 @@
     <xacro:property name="ODM_joint_type" value="fixed"/>
     <!-- import main body description -->
-    <xacro:include filename="$(find neo_simulation2)/robots/mmo_700/urdf/mmo_700_body.urdf.xacro"/>
+    <xacro:include filename="$(find steve_simulation)/robots/mmo_700/urdf/mmo_700_body.urdf.xacro"/>
     <!-- If Simulation is used -->
     <xacro:if value="$(arg use_gazebo)">
-        <xacro:include filename="$(find neo_simulation2)/robots/mmo_700/urdf/mmo_700_gazebo.urdf.xacro"/>
+        <xacro:include filename="$(find steve_simulation)/robots/mmo_700/urdf/mmo_700_gazebo.urdf.xacro"/>
     </xacro:if>
     <!-- Check if one of the arms is used -->
@@ -34,5 +34,5 @@
     <xacro:if value="${use_arm}">
         <!-- cabinet -->
-        <xacro:include filename="$(find neo_simulation2)/components/common_macro/mpo_cabinet_macro.xacro"/>
+        <xacro:include filename="$(find steve_simulation)/components/common_macro/mpo_cabinet_macro.xacro"/>
         <xacro:cabinet
             neo_robot_name="mmo_700"
@@ -47,13 +47,13 @@
         <!-- Universal Robotics Arm-->
         <xacro:if value="${arm == 'ur5' or arm == 'ur10' or arm == 'ur5e' or arm == 'ur10e'}">
-            <xacro:include filename="$(find neo_simulation2)/components/arm/ur_arm.urdf.xacro"/>
+            <xacro:include filename="$(find steve_simulation)/components/arm/ur_arm.urdf.xacro"/>
         </xacro:if>
         <!-- Elite Arm -->
         <xacro:if value="${arm == 'ec66' or arm == 'cs66'}">
-            <xacro:include filename="$(find neo_simulation2)/components/arm/elite_arm.urdf.xacro"/>
+            <xacro:include filename="$(find steve_simulation)/components/arm/elite_arm.urdf.xacro"/>
         </xacro:if>
         <!-- Wrist camera is now integrated into ur_arm assembly (with dummy end-effector) -->
         <!-- <xacro:if value="$(arg include_wrist_camera)">
-            <xacro:include filename="$(find neo_simulation2)/components/cameras/wrist_d405.urdf.xacro"/>
+            <xacro:include filename="$(find steve_simulation)/components/cameras/wrist_d405.urdf.xacro"/>
             <xacro:wrist_d405 parent="ur5etool0" use_gazebo="$(arg use_gazebo)"/>
         </xacro:if> -->
@@ -61,5 +61,5 @@
     <!-- Optional depth camera on base -->
     <xacro:if value="$(arg include_depth_camera)">
-        <xacro:include filename="$(find neo_simulation2)/robots/mmo_700/urdf/macro/depth_camera_macro.xacro"/>
+        <xacro:include filename="$(find steve_simulation)/robots/mmo_700/urdf/macro/depth_camera_macro.xacro"/>
         <xacro:depth_camera name="front_camera" parent="base_link" use_gazebo="$(arg use_gazebo)">
             <origin xyz="0.292 0 0.716" rpy="0 0 0"/>
@@ -68,5 +68,5 @@
     <!-- Pan-tilt camera tower on base -->
     <xacro:if value="$(arg include_pan_tilt)">
-        <xacro:include filename="$(find neo_simulation2)/components/pan_tilt/pan_tilt_tower.urdf.xacro"/>
+        <xacro:include filename="$(find steve_simulation)/components/pan_tilt/pan_tilt_tower.urdf.xacro"/>
         <xacro:pan_tilt_tower parent_link="base_link" use_gazebo="$(arg use_gazebo)"/>
     </xacro:if>

File: robots/mmo_700/mmo_700_processed.urdf (robot description, URDF)
Before this commit: robot mmo_700, 42 links, 41 joints
Links:
- link base_link: geometry collision mesh filename=package://steve_simulation/robots/mmo_700/meshes/MPO-700-BO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 scale=0.001 0.001 0.001; visual mesh filename=package://steve_simulation/robots/mmo_700/meshes/MPO-700-BO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 scale=0.001 0.001 0.001
- link cabinet_link: geometry collision mesh filename=package://steve_simulation/robots/mpo_700/meshes/cabin.dae scale=0.001 0.001 0.001; visual mesh filename=package://steve_simulation/robots/mmo_700/meshes/cabin.dae scale=0.001 0.001 0.001
- link lidar_1_link: geometry collision mesh filename=package://steve_simulation/components/meshes/SICK-S300.dae scale=0.001 0.001 0.001; visual mesh filename=package://steve_simulation/components/meshes/SICK-S300.dae scale=0.001 0.001 0.001
- link lidar_2_link: geometry collision mesh filename=package://steve_simulation/components/meshes/SICK-S300.dae scale=0.001 0.001 0.001; visual mesh filename=package://steve_simulation/components/meshes/SICK-S300.dae scale=0.001 0.001 0.001
- link mpo_700_caster_back_left_link: geometry collision mesh filename=package://steve_simulation/robots/mpo_700/meshes/MPO-700-HE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 scale=0.001 0.001 0.001; visual mesh filename=package://steve_simulation/robots/mpo_700/meshes/MPO-700-HE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 scale=0.001 0.001 0.001
- link mpo_700_caster_back_right_link: geometry collision mesh filename=package://steve_simulation/robots/mpo_700/meshes/MPO-700-HE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 scale=0.001 0.001 0.001; visual mesh filename=package://steve_simulation/robots/mpo_700/meshes/MPO-700-HE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 scale=0.001 0.001 0.001
- link mpo_700_caster_front_left_link: geometry collision mesh filename=package://steve_simulation/robots/mpo_700/meshes/MPO-700-HE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 scale=0.001 0.001 0.001; visual mesh filename=package://steve_simulation/robots/mpo_700/meshes/MPO-700-HE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 scale=0.001 0.001 0.001
- link mpo_700_caster_front_right_link: geometry collision mesh filename=package://steve_simulation/robots/mpo_700/meshes/MPO-700-HE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 scale=0.001 0.001 0.001; visual mesh filename=package://steve_simulation/robots/mpo_700/meshes/MPO-700-HE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 scale=0.001 0.001 0.001
- link mpo_700_wheel_back_left_link: geometry collision sphere radius=0.09; visual mesh filename=package://steve_simulation/robots/mpo_700/meshes/MPO-700-WH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 scale=0.001 0.001 0.001
- link mpo_700_wheel_back_right_link: geometry collision sphere radius=0.09; visual mesh filename=package://steve_simulation/robots/mpo_700/meshes/MPO-700-WH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 scale=0.001 0.001 0.001
- link mpo_700_wheel_front_left_link: geometry collision sphere radius=0.09; visual mesh filename=package://steve_simulation/robots/mpo_700/meshes/MPO-700-WH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 scale=0.001 0.001 0.001
- link mpo_700_wheel_front_right_link: geometry collision sphere radius=0.09; visual mesh filename=package://steve_simulation/robots/mpo_700/meshes/MPO-700-WH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 scale=0.001 0.001 0.001
- link wrist_camera_link: geometry collision box size=0.025 0.090 0.023; visual mesh filename=package://steve_simulation/robots/mmo_700/meshes/cameras/d4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 scale=0.001 0.001 0.001
- link wrist_d405_mount: geometry collision box size=0.02 0.09 0.025; visual mesh filename=package://steve_simulation/robots/mmo_700/meshes/cameras/d4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 scale=0.001 0.001 0.001

File: robots/mmo_700/urdf/macro/cabinet.xacro (robot description, xacro)
@@ -19,5 +19,5 @@
         <origin xyz="0 0 0" rpy="0 0 -1.5708" />
         <geometry>
-            <mesh filename="package://neo_simulation2/robots/mmo_700/meshes/cabin.dae" scale="0.001 0.001 0.001"/>
+            <mesh filename="package://steve_simulation/robots/mmo_700/meshes/cabin.dae" scale="0.001 0.001 0.001"/>
         </geometry>
       </visual>
@@ -25,5 +25,5 @@
         <origin xyz="0 0 0" rpy="0 0 -1.5708" />
         <geometry>
-            <mesh filename="package://neo_simulation2/robots/mmo_700/meshes/cabin.dae" scale="0.001 0.001 0.001"/>
+            <mesh filename="package://steve_simulation/robots/mmo_700/meshes/cabin.dae" scale="0.001 0.001 0.001"/>
         </geometry>
       </collision>

File: robots/mmo_700/urdf/macro/micro_scan.xacro (robot description, xacro)
@@ -17,5 +17,5 @@
         <origin xyz="0 0 -0.06" rpy="1.57 0 0" />
       <geometry>
-        <mesh filename="package://neo_simulation2/robots/mpo_700/meshes/SICK-MICROSCAN3.dae" scale="0.001 0.001 0.001" />
+        <mesh filename="package://steve_simulation/robots/mpo_700/meshes/SICK-MICROSCAN3.dae" scale="0.001 0.001 0.001" />
         </geometry>
       </visual>
@@ -23,5 +23,5 @@
         <origin xyz="0 0 -0.06" rpy="1.57 0 0" />
         <geometry>
-          <mesh filename="package://neo_simulation2/robots/mpo_700/meshes/SICK-MICROSCAN3.dae" scale="0.001 0.001 0.001" />
+          <mesh filename="package://steve_simulation/robots/mpo_700/meshes/SICK-MICROSCAN3.dae" scale="0.001 0.001 0.001" />
         </geometry>
       </collision>

File: robots/mmo_700/urdf/macro/mpo_700_body.xacro (robot description, xacro)
@@ -13,5 +13,5 @@
         <origin xyz="0.0 0.0 0.0" rpy="0 0 -1.571" />
         <geometry>
-            <mesh filename="package://neo_simulation2/robots/mmo_700/meshes/MPO-700-BODY.dae" scale="0.001 0.001 0.001"/>
+            <mesh filename="package://steve_simulation/robots/mmo_700/meshes/MPO-700-BODY.dae" scale="0.001 0.001 0.001"/>
         </geometry>
       </visual>
@@ -19,5 +19,5 @@
         <origin xyz="0. 0. 0." rpy="0 0 -1.571" />
         <geometry>
-            <mesh filename="package://neo_simulation2/robots/mmo_700/meshes/MPO-700-BODY.dae" scale="0.001 0.001 0.001"/>
+            <mesh filename="package://steve_simulation/robots/mmo_700/meshes/MPO-700-BODY.dae" scale="0.001 0.001 0.001"/>
         </geometry>
       </collision>

File: robots/mmo_700/urdf/macro/mpo_700_caster.xacro (robot description, xacro)
@@ -19,5 +19,5 @@
      <origin xyz="0 0 0.10" rpy="0 0 0"/>
      <geometry>
-        <mesh filename="package://neo_simulation2/robots/mmo_700/meshes/MPO-700-HEAD.dae" scale="0.001 0.001 0.001"/>
+        <mesh filename="package://steve_simulation/robots/mmo_700/meshes/MPO-700-HEAD.dae" scale="0.001 0.001 0.001"/>
      </geometry>
     </visual>
@@ -25,5 +25,5 @@
      <origin xyz="0 0 0.10" rpy="0 0 0" />
      <geometry>
-        <mesh filename="package://neo_simulation2/robots/mmo_700/meshes/MPO-700-HEAD.dae" scale="0.001 0.001 0.001"/>
+        <mesh filename="package://steve_simulation/robots/mmo_700/meshes/MPO-700-HEAD.dae" scale="0.001 0.001 0.001"/>
      </geometry>
     </collision>
@@ -47,5 +47,5 @@
      <origin xyz="0 0 0.10" rpy="0 0 0"/>
      <geometry>
-        <mesh filename="package://neo_simulation2/robots/mmo_700/meshes/MPO-700-HEAD.dae" scale="0.001 0.001 0.001"/>
+        <mesh filename="package://steve_simulation/robots/mmo_700/meshes/MPO-700-HEAD.dae" scale="0.001 0.001 0.001"/>
      </geometry>
     </visual>
@@ -53,5 +53,5 @@
      <origin xyz="0 0 0.10" rpy="0 0 0" />
      <geometry>
-        <mesh filename="package://neo_simulation2/robots/mmo_700/meshes/MPO-700-HEAD.dae" scale="0.001 0.001 0.001"/>
+        <mesh filename="package://steve_simulation/robots/mmo_700/meshes/MPO-700-HEAD.dae" scale="0.001 0.001 0.001"/>
      </geometry>
     </collision>
@@ -75,5 +75,5 @@
      <origin xyz="0 0 0.10" rpy="0 0 0"/>
      <geometry>
-        <mesh filename="package://neo_simulation2/robots/mmo_700/meshes/MPO-700-HEAD.dae" scale="0.001 0.001 0.001"/>
+        <mesh filename="package://steve_simulation/robots/mmo_700/meshes/MPO-700-HEAD.dae" scale="0.001 0.001 0.001"/>
      </geometry>
     </visual>
@@ -81,5 +81,5 @@
      <origin xyz="0 0 0.10" rpy="0 0 0" />
      <geometry>
-        <mesh filename="package://neo_simulation2/robots/mmo_700/meshes/MPO-700-HEAD.dae" scale="0.001 0.001 0.001"/>
+        <mesh filename="package://steve_simulation/robots/mmo_700/meshes/MPO-700-HEAD.dae" scale="0.001 0.001 0.001"/>
      </geometry>
     </collision>
@@ -103,5 +103,5 @@
      <origin xyz="0 0 0.10" rpy="0 0 0"/>
      <geometry>
-        <mesh filename="package://neo_simulation2/robots/mmo_700/meshes/MPO-700-HEAD.dae" scale="0.001 0.001 0.001"/>
+        <mesh filename="package://steve_simulation/robots/mmo_700/meshes/MPO-700-HEAD.dae" scale="0.001 0.001 0.001"/>
      </geometry>
     </visual>
@@ -109,5 +109,5 @@
      <origin xyz="0 0 0.10" rpy="0 0 0" />
      <geometry>
-        <mesh filename="package://neo_simulation2/robots/mmo_700/meshes/MPO-700-HEAD.dae" scale="0.001 0.001 0.001"/>
+        <mesh filename="package://steve_simulation/robots/mmo_700/meshes/MPO-700-HEAD.dae" scale="0.001 0.001 0.001"/>
      </geometry>
     </collision>

File: robots/mmo_700/urdf/macro/mpo_700_wheel.xacro (robot description, xacro)
@@ -20,5 +20,5 @@
      <origin xyz="0 0 0" rpy="0 0 0"/>
      <geometry>
-        <mesh filename="package://neo_simulation2/robots/mmo_700/meshes/MPO-700-WHEEL.dae" scale="0.001 0.001 0.001"/>
+        <mesh filename="package://steve_simulation/robots/mmo_700/meshes/MPO-700-WHEEL.dae" scale="0.001 0.001 0.001"/>
      </geometry>
     </visual>
@@ -26,5 +26,5 @@
      <origin xyz="0 0 0" rpy="0 0 0" />
      <geometry>
-        <mesh filename="package://neo_simulation2/robots/mmo_700/meshes/MPO-700-WHEEL.dae" scale="0.001 0.001 0.001"/>
+        <mesh filename="package://steve_simulation/robots/mmo_700/meshes/MPO-700-WHEEL.dae" scale="0.001 0.001 0.001"/>
      </geometry>
     </collision>

File: robots/mmo_700/urdf/macro/sick_S300.xacro (robot description, xacro)
@@ -17,5 +17,5 @@
         <origin xyz="0 0 -0.12" rpy="-1.57 0 3.14" />
         <geometry>
-        <mesh filename="package://neo_simulation2/components/meshes/SICK-S300.dae" scale="0.001 0.001 0.001" />
+        <mesh filename="package://steve_simulation/components/meshes/SICK-S300.dae" scale="0.001 0.001 0.001" />
         </geometry>
       </visual>
@@ -23,5 +23,5 @@
         <origin xyz="0 0 -0.12" rpy="-1.57 0 3.14" />
         <geometry>
-        <mesh filename="package://neo_simulation2/components/meshes/SICK-S300.dae" scale="0.001 0.001 0.001" />
+        <mesh filename="package://steve_simulation/components/meshes/SICK-S300.dae" scale="0.001 0.001 0.001" />
         </geometry>
       </collision>
