Commit message: Restructure

File: robots/mmo_700/urdf/mmo_700_body.urdf.xacro (robot description, xacro)
@@ -11,5 +11,5 @@
             <origin rpy="0 0 -1.571" xyz="0.0 0.0 0.0"/>
             <geometry>
-                <mesh filename="package://neo_simulation2/robots/mmo_700/meshes/MPO-700-BODY.dae" scale="0.001 0.001 0.001"/>
+                <mesh filename="package://steve_simulation/robots/mmo_700/meshes/MPO-700-BODY.dae" scale="0.001 0.001 0.001"/>
             </geometry>
         </visual>
@@ -17,5 +17,5 @@
             <origin rpy="0 0 -1.571" xyz="0. 0. 0."/>
             <geometry>
-                <mesh filename="package://neo_simulation2/robots/mmo_700/meshes/MPO-700-BODY.dae" scale="0.001 0.001 0.001"/>
+                <mesh filename="package://steve_simulation/robots/mmo_700/meshes/MPO-700-BODY.dae" scale="0.001 0.001 0.001"/>
             </geometry>
         </collision>
@@ -45,5 +45,5 @@
             <origin rpy="-1.57 0 3.14" xyz="0 0 -0.12"/>
             <geometry>
-                <mesh filename="package://neo_simulation2/components/meshes/SICK-S300.dae" scale="0.001 0.001 0.001"/>
+                <mesh filename="package://steve_simulation/components/meshes/SICK-S300.dae" scale="0.001 0.001 0.001"/>
             </geometry>
         </visual>
@@ -51,5 +51,5 @@
             <origin rpy="-1.57 0 3.14" xyz="0 0 -0.12"/>
             <geometry>
-                <mesh filename="package://neo_simulation2/components/meshes/SICK-S300.dae" scale="0.001 0.001 0.001"/>
+                <mesh filename="package://steve_simulation/components/meshes/SICK-S300.dae" scale="0.001 0.001 0.001"/>
             </geometry>
         </collision>
@@ -71,5 +71,5 @@
             <origin rpy="-1.57 0 3.14" xyz="0 0 -0.12"/>
             <geometry>
-                <mesh filename="package://neo_simulation2/components/meshes/SICK-S300.dae" scale="0.001 0.001 0.001"/>
+                <mesh filename="package://steve_simulation/components/meshes/SICK-S300.dae" scale="0.001 0.001 0.001"/>
             </geometry>
         </visual>
@@ -77,11 +77,11 @@
             <origin rpy="-1.57 0 3.14" xyz="0 0 -0.12"/>
             <geometry>
-                <mesh filename="package://neo_simulation2/components/meshes/SICK-S300.dae" scale="0.001 0.001 0.001"/>
+                <mesh filename="package://steve_simulation/components/meshes/SICK-S300.dae" scale="0.001 0.001 0.001"/>
             </geometry>
         </collision>
     </link>
     <!-- Import wheel macros from MPO_700 (same platform) -->
-    <xacro:include filename="$(find neo_simulation2)/robots/mmo_700/urdf/macro/mpo_700_wheel.xacro"/>
-    <xacro:include filename="$(find neo_simulation2)/robots/mmo_700/urdf/macro/mpo_700_caster.xacro"/>
+    <xacro:include filename="$(find steve_simulation)/robots/mmo_700/urdf/macro/mpo_700_wheel.xacro"/>
+    <xacro:include filename="$(find steve_simulation)/robots/mmo_700/urdf/macro/mpo_700_caster.xacro"/>
     <!-- Caster wheels -->
     <xacro:mpo_700_caster_0

File: robots/mmo_700/urdf/mmo_700_gazebo.urdf.xacro (robot description, xacro)
@@ -2,6 +2,6 @@
 <robot xmlns:xacro="http://www.ros.org/wiki/xacro" name="mmo_700">
     <!-- Include macros from common components -->
-    <xacro:include filename="$(find neo_simulation2)/components/common_macro/gazebo_lidar_macro.xacro" />
-    <xacro:include filename="$(find neo_simulation2)/components/common_macro/gazebo_object_controller_macro.xacro" />
+    <xacro:include filename="$(find steve_simulation)/components/common_macro/gazebo_lidar_macro.xacro" />
+    <xacro:include filename="$(find steve_simulation)/components/common_macro/gazebo_object_controller_macro.xacro" />
     <!-- Properties -->
     <xacro:property name="lidar_1_update_rate" value="40" />
