Commit message: Camera Fix

File: components/cameras/l515_simplified.urdf.xacro (robot description, xacro)
@@ -35,12 +35,11 @@
     <!-- Color optical frame -->
     <joint name="${name}_color_optical_joint" type="fixed">
-      <origin xyz="0 0 0" rpy="${-M_PI/2} 0 ${-M_PI/2}"/>
+      <origin xyz="0 0 0.01" rpy="0 -1.57 1.57"/>
       <parent link="${name}_link"/>
       <child link="${name}_color_optical_frame"/>
     </joint>
     <link name="${name}_color_optical_frame"/>
-    <!-- Depth optical frame -->
     <joint name="${name}_depth_optical_joint" type="fixed">
-      <origin xyz="0 0 0" rpy="${-M_PI/2} 0 ${-M_PI/2}"/>
+      <origin xyz="0 0 0.01" rpy="0 -1.57 1.57"/>
       <parent link="${name}_link"/>
       <child link="${name}_depth_optical_frame"/>
@@ -49,5 +48,5 @@
     <!-- Gazebo depth camera plugin for ROS2 -->
     <xacro:if value="${use_gazebo}">
-      <gazebo reference="${name}_link">
+      <gazebo reference="${name}_color_optical_frame">
         <sensor name="${name}" type="depth">
           <update_rate>30</update_rate>

File: components/cameras/wrist_d405.urdf.xacro (robot description, xacro)
@@ -39,5 +39,5 @@
 <link name="wrist_camera_link">
   <visual>
-    <origin xyz="0 0 0" rpy="0 0 0"/>
+    <origin xyz="0.01 0 0.01" rpy="0 1.57 0"/>
     <geometry>
       <mesh filename="package://neo_simulation2/robots/mmo_700/meshes/cameras/d405/d405.stl" scale="0.001 0.001 0.001"/>

File: components/common_macro/mpo_cabinet_macro.xacro (robot description, xacro)
@@ -32,5 +32,5 @@
                 <origin rpy="${collision_rpy}" xyz="0 0 0"/>
                 <geometry>
-                    <mesh filename="package://neo_simulation2/robots/mpo_700/meshes/cabin.dae" scale="${model_scale}"/>
+                    <mesh filename="package://neo_simulation2/robots/${neo_robot_name}/meshes/cabin.dae" scale="${model_scale}"/>
                 </geometry>
             </collision>

File: components/pan_tilt/pan_tilt_tower.urdf.xacro (robot description, xacro)
@@ -42,11 +42,11 @@
     <xacro:pan_tilt_ros2_control name="pan_tilt"/>
     <!-- Include L515 camera macro -->
-    <xacro:include filename="$(find neo_simulation2)/components/realsense/l515_simplified.urdf.xacro"/>
-    <!-- L515 Camera mounted on tilt bracket -->
+    <xacro:include filename="$(find neo_simulation2)/components/cameras/l515_simplified.urdf.xacro"/>
+    <!-- L515 Camera mounted on pan bracket (follows both pan and tilt) -->
     <xacro:sensor_l515_simplified
-      parent="pan_tilt_tilt_bracket_link"
+      parent="pan_tilt_pan_bracket_link"
       name="pan_tilt_camera"
       use_gazebo="${use_gazebo}">
-      <origin xyz="0 0.0423 -0.028" rpy="0 0 ${pi/2}"/>
+      <origin xyz="0 0.04 0" rpy="0 ${pi/2} ${pi/2}"/>
     </xacro:sensor_l515_simplified>
     <!-- Gazebo materials -->

File: robots/mmo_700/urdf/macro/cabinet.xacro (robot description, xacro)
@@ -19,5 +19,5 @@
         <origin xyz="0 0 0" rpy="0 0 -1.5708" />
         <geometry>
-            <mesh filename="package://neo_simulation2/robots/mmo_500/meshes/cabin.dae" scale="0.001 0.001 0.001"/>
+            <mesh filename="package://neo_simulation2/robots/mmo_700/meshes/cabin.dae" scale="0.001 0.001 0.001"/>
         </geometry>
       </visual>
@@ -25,5 +25,5 @@
         <origin xyz="0 0 0" rpy="0 0 -1.5708" />
         <geometry>
-            <mesh filename="package://neo_simulation2/robots/mmo_500/meshes/cabin.dae" scale="0.001 0.001 0.001"/>
+            <mesh filename="package://neo_simulation2/robots/mmo_700/meshes/cabin.dae" scale="0.001 0.001 0.001"/>
         </geometry>
       </collision>

File: robots/mmo_700/urdf/macro/sick_S300.xacro (robot description, xacro)
@@ -17,5 +17,5 @@
         <origin xyz="0 0 -0.12" rpy="-1.57 0 3.14" />
         <geometry>
-        <mesh filename="package://neo_simulation2/robots/mpo_700/meshes/SICK-S300.dae" scale="0.001 0.001 0.001" />
+        <mesh filename="package://neo_simulation2/components/meshes/SICK-S300.dae" scale="0.001 0.001 0.001" />
         </geometry>
       </visual>
@@ -23,5 +23,5 @@
         <origin xyz="0 0 -0.12" rpy="-1.57 0 3.14" />
         <geometry>
-        <mesh filename="package://neo_simulation2/robots/mpo_700/meshes/SICK-S300.dae" scale="0.001 0.001 0.001" />
+        <mesh filename="package://neo_simulation2/components/meshes/SICK-S300.dae" scale="0.001 0.001 0.001" />
         </geometry>
       </collision>
