Commit message: Update URDF and navigation config

File: components/dynamixel/dynamixel_motor_xl-430.urdf.xacro (robot description, xacro)
@@ -36,4 +36,5 @@
         <axis xyz="${motor_direction} 0 0"/>
         <limit effort="1.5" lower="-${M_PI / 180 * 110}" upper="${M_PI / 180 * 110}" velocity="6.178465545"/>
+        <dynamics damping="0.7" friction="0.5"/>
       </joint>
     </xacro:if>
@@ -45,4 +46,5 @@
         <axis xyz="${motor_direction} 0 0"/>
         <limit effort="1.5" lower="-${M_PI / 180 * 180}" upper="${M_PI / 180 * 20}" velocity="6.178465545"/>
+        <dynamics damping="0.7" friction="0.5"/>
       </joint>
     </xacro:if>

File: components/pan_tilt/pan_tilt.ros2_control.xacro (robot description, xacro)
@@ -11,5 +11,7 @@
           <param name="max">3.14</param>
         </command_interface>
-        <state_interface name="position"/>
+        <state_interface name="position">
+          <param name="initial_value">0.0</param>
+        </state_interface>
         <state_interface name="velocity"/>
       </joint>
@@ -19,5 +21,7 @@
           <param name="max">3.14</param>
         </command_interface>
-        <state_interface name="position"/>
+        <state_interface name="position">
+          <param name="initial_value">-0.2</param>
+        </state_interface>
         <state_interface name="velocity"/>
       </joint>
