Commit message: Add Pantilt

File: components/pan_tilt/pan_tilt_tower.urdf.xacro (robot description, xacro)
@@ -41,71 +41,13 @@
     <xacro:include filename="$(find neo_simulation2)/components/pan_tilt/pan_tilt.ros2_control.xacro"/>
     <xacro:pan_tilt_ros2_control name="pan_tilt"/>
-    <!-- Camera with D435 mesh - EXACT steve mounting position -->
-    <joint name="pan_tilt_camera_joint" type="fixed">
-      <parent link="pan_tilt_tilt_bracket_link"/>
-      <child link="pan_tilt_camera_link"/>
+    <!-- Include L515 camera macro -->
+    <xacro:include filename="$(find neo_simulation2)/components/realsense/l515_simplified.urdf.xacro"/>
+    <!-- L515 Camera mounted on tilt bracket -->
+    <xacro:sensor_l515_simplified
+      parent="pan_tilt_tilt_bracket_link"
+      name="pan_tilt_camera"
+      use_gazebo="${use_gazebo}">
       <origin xyz="0 0.0423 -0.028" rpy="0 0 ${pi/2}"/>
-    </joint>
-    <link name="pan_tilt_camera_link">
-      <visual>
-        <origin xyz="0 0 0" rpy="0 0 0"/>
-        <geometry>
-          <mesh filename="package://neo_simulation2/robots/mmo_700/meshes/cameras/d435/d435.dae" scale="1 1 1"/>
-        </geometry>
-      </visual>
-      <collision>
-        <origin xyz="0 0 0" rpy="0 0 0"/>
-        <geometry>
-          <box size="0.09 0.025 0.025"/>
-        </geometry>
-      </collision>
-      <inertial>
-        <mass value="0.072"/>
-        <origin xyz="0 0 0" rpy="0 0 0"/>
-        <inertia ixx="0.0001" ixy="0" ixz="0" iyy="0.0001" iyz="0" izz="0.0001"/>
-      </inertial>
-    </link>
-    <!-- Camera optical frames -->
-    <joint name="pan_tilt_camera_optical_joint" type="fixed">
-      <origin xyz="0 0 0" rpy="${-pi/2} 0 ${-pi/2}"/>
-      <parent link="pan_tilt_camera_link"/>
-      <child link="pan_tilt_camera_optical_frame"/>
-    </joint>
-    <link name="pan_tilt_camera_optical_frame"/>
-    <!-- Gazebo depth camera plugin -->
-    <xacro:if value="${use_gazebo}">
-      <gazebo reference="pan_tilt_camera_link">
-        <sensor name="pan_tilt_camera" type="depth">
-          <update_rate>30</update_rate>
-          <camera>
-            <horizontal_fov>${70*pi/180}</horizontal_fov>
-            <image>
-              <width>640</width>
-              <height>480</height>
-              <format>R8G8B8</format>
-            </image>
-            <clip>
-              <near>0.1</near>
-              <far>9.0</far>
-            </clip>
-          </camera>
-          <plugin name="pan_tilt_camera_controller" filename="libgazebo_ros_camera.so">
-            <ros>
-              <namespace>pan_tilt_camera</namespace>
-              <remapping>image_raw:=color/image_raw</remapping>
-              <remapping>camera_info:=color/camera_info</remapping>
-              <remapping>depth/image_raw:=aligned_depth_to_color/image_raw</remapping>
-              <remapping>depth/camera_info:=aligned_depth_to_color/camera_info</remapping>
-              <remapping>points:=depth/color/points</remapping>
-            </ros>
-            <camera_name>pan_tilt_camera</camera_name>
-            <frame_name>pan_tilt_camera_optical_frame</frame_name>
-            <hack_baseline>0.05</hack_baseline>
-            <min_depth>0.1</min_depth>
-            <max_depth>9.0</max_depth>
-          </plugin>
-        </sensor>
-      </gazebo>
-    </xacro:if>
+    </xacro:sensor_l515_simplified>
     <!-- Gazebo materials -->
     <xacro:if value="${use_gazebo}">

Commit message: Fix Camera Frame

File: components/pan_tilt/pan_tilt_tower.urdf.xacro (robot description, xacro)
@@ -48,5 +48,5 @@
       name="pan_tilt_camera"
       use_gazebo="${use_gazebo}">
-      <origin xyz="0 0.04 0" rpy="0 ${pi/2} ${pi/2}"/>
+      <origin xyz="0 0.04 0" rpy="0 ${pi/2} 0"/>
     </xacro:sensor_l515_simplified>
     <!-- Gazebo materials -->

Commit message: Camera Fix Mesh

File: components/pan_tilt/pan_tilt_tower.urdf.xacro (robot description, xacro)
@@ -48,5 +48,5 @@
       name="pan_tilt_camera"
       use_gazebo="${use_gazebo}">
-      <origin xyz="0 0.04 0" rpy="0 ${pi/2} 0"/>
+      <origin xyz="0 0.04 0" rpy="${pi/2} ${pi/2} 0"/>
     </xacro:sensor_l515_simplified>
     <!-- Gazebo materials -->

Commit message: ROBOT URDF FIXXXXX cd src/neo_simulation2/cd src/neo_simulation2/!

File: components/pan_tilt/pan_tilt_tower.urdf.xacro (robot description, xacro)
@@ -48,5 +48,5 @@
       name="pan_tilt_camera"
       use_gazebo="${use_gazebo}">
-      <origin xyz="0 0.04 0" rpy="${pi/2} ${pi/2} 0"/>
+      <origin xyz="0 0.04 0" rpy="${pi/2} ${pi/2} ${pi}"/>
     </xacro:sensor_l515_simplified>
     <!-- Gazebo materials -->
